File: hardware/obd_tracker_carrier_v1/obd_tracker_carrier_v1.kicad_pcb (KiCad board)
At the start: 2 copper layers, 88 x 40 mm, 47 parts, among them J1 OBD2 harness 12V/GND/CANH/CANL, J2 JST-PH-2 LiPo, populate inste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, J3A T-SIM7000G low profile header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, J3B T-SIM7000G low profile header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, U2 TPS54360DDAR 12V-to-5V buck, U3 TJA1051T/3 5V CAN transceiver, U4 ADXL375BCCZ-RL7

Commit message: v0.11.4 — post at 10s whenever the engine is running (OBD rpm), not just moving
The live vitals dash felt laggy while idling because posting cadence
was driven by GPS motion: an engine idling in place isn't a 'trip', so
the tracker dropped to the 2-min parked cadence even as OBD values
changed every second. OBD rpm is a real engine-on signal (which GPS
motion never was), so nextIntervalMs now posts at 10s whenever the
engine is confirmed running — idling or driving. Bounded to actual
engine-on time and cheap over UDP; highway still uses the 5s branch.

Co-Authored-By: Claude Fable 5 <noreply@anthropic.com>
Connections:
- U2 pad 5: GND -> BUCK_FB
- U2 pad 7: BUCK_FB -> GND
- U4 pad 1: GND -> +3V3
- U4 pad 12: (no net) -> GND
- U4 pad 13: GND -> I2C_SDA_GPIO21
- U4 pad 14: GND -> I2C_SCL_GPIO22
- U4 pad 2: +3V3 -> GND
- U4 pad 4: I2C_SCL_GPIO22 -> GND
- U4 pad 5: I2C_SDA_GPIO21 -> GND
- U4 pad 6: ACCEL_INT1_GPIO34 -> +3V3
- U4 pad 7: (no net) -> +3V3
- U4 pad 8: +3V3 -> ACCEL_INT1_GPIO34
- U4 pad 9: GND -> (no net)
Routing:
- net VBAT: track 77.0 -> 252.4 mm
- net +3V3: track 0.00 -> 147.0 mm
- net VIN_PROT: track 9.66 -> 45.0 mm
- net +5V: track 40.7 -> 71.3 mm
- net BUCK_FB: track 0.00 -> 20.0 mm
- net ACCEL_INT1_GPIO34: track 60.1 -> 79.1 mm
- net GND: track 16.8 -> 0.00 mm
- net BUCK_SW: track 0.00 -> 15.9 mm
- net VEH_SENSE_GPIO35: track 14.7 -> 27.3 mm
- net CANH: track 34.6 -> 47.1 mm
- net CANL: track 34.6 -> 46.7 mm
- net VBAT_SENSE_GPIO36: track 28.2 -> 39.8 mm
- net CAN_RX_GPIO33: track 40.6 -> 51.1 mm
- net VIN_FUSED: track 4.60 -> 14.7 mm
- net CAN_TX_GPIO32: track 40.3 -> 49.8 mm
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